File: test_boards/pcb/transducer.kicad_sch (KiCad schematic)
At the start: 8 parts, among them Q1 SI2324A-TP, Q2 SI2324A-TP, U1 EG2131D

Commit message: w
Parts:
- C1, C2, C3, D1: Vendor (none) -> Digi-Key
- LS1: footprint (none) -> Footprints:Ultrasonic_Transducer_D16mm_H7mm_P10mm; Vendor (none) -> LCSC
- Q1, Q2: value SI2324A-TP -> G2003A; footprint Package_TO_SOT_SMD:SOT-23 -> Package_TO_SOT_SMD:SOT-23-3; Manufacturer Part Number (none) -> G2003A; Vendor (none) -> Digi-Key; Vendor Part Number (none) -> 3141-G2003ACT-ND
- U1: Vendor (none) -> LCSC
Other:
- note removed: "Higher Vds MOSFETS?"
- note removed: "capacitor should be 10-15 times Qg / Vgd"
- moved on the sheet: C1

Commit message: w
Parts:
- renumbered C2 to C7, C1 to C8, C3 to C9, U1 to U5

Commit message: w
Parts:
- added R39, R63: 10kΩ, Resistor_SMD:R_0402_1005Metric, symbol Device:R_US
Connections:
- net HIN: now also R39.2; no longer U5.2 (HIN)
- net ~{LIN}: now also R63.1; no longer U5.3 (~{LIN})
- new net HIN_IN: R39.1, U5.2 (HIN)
- new net ~{LIN_IN}: R63.2, U5.3 (~{LIN})

Commit message: w
Parts:
- added R132, R90: 10kΩ, Resistor_SMD:R_0402_1005Metric, symbol Device:R_US
- D1: value SUF4007 -> ES1DF; footprint Diode_SMD:D_MELF -> Diode_SMD:D_SMA; Manufacturer Part Number (none) -> ES1DF; Vendor Part Number (none) -> 5399-ES1DFCT-ND
- LS1: value Speaker_Ultrasound -> 40kHz
Connections:
- net GND: now also R132.1, R90.2
- net HIN: now also R90.1
- net ~{LIN}: now also R132.2
