File: test_boards/pcb/transducer_rx.kicad_sch (KiCad schematic)
At the start: 17 parts, among them U3 LOG300RGT, U5 OPA388xxDBV

Commit message: w
Parts:
- added R32: 10Ω, Resistor_SMD:R_0603_1608Metric_Pad0.98x0.95mm_HandSolder, symbol Device:R_US
- C10, C8, C9: footprint (none) -> Capacitor_SMD:C_0402_1005Metric; Vendor (none) -> Digi-Key
- C11, C12: value 1μF -> 1nF; footprint Capacitor_SMD:C_1206_3216Metric -> Capacitor_SMD:C_0402_1005Metric; Vendor (none) -> Digi-Key
- C4: value 1μF -> 22nF; footprint Capacitor_SMD:C_1206_3216Metric -> Capacitor_SMD:C_0805_2012Metric; Manufacturer Part Number (none) -> C0805C223K5GEC7210; Vendor (none) -> Digi-Key; Vendor Part Number (none) -> 399-C0805C223K5GEC7210CT-ND
- C5: value 10nF -> 100nF; footprint (none) -> Capacitor_SMD:C_0603_1608Metric; Vendor (none) -> Digi-Key
- C6: value 1μF -> 100μF; footprint (none) -> Capacitor_Tantalum_SMD:CP_EIA-7343-31_Kemet-D; symbol Device:C -> Device:C_Polarized_US; Manufacturer Part Number (none) -> TAJD107K016SNJV; Vendor (none) -> Digi-Key; Vendor Part Number (none) -> 478-TAJD107K016SNJVCT-ND
- C7: footprint (none) -> Capacitor_SMD:C_0603_1608Metric; Vendor (none) -> Digi-Key
- LS2: footprint (none) -> Footprints:Ultrasonic_Transducer_D16mm_H7mm_P10mm; Vendor (none) -> LCSC
- R1, R2, R3, R4, R5: footprint (none) -> Resistor_SMD:R_0402_1005Metric; Vendor (none) -> Digi-Key
- U3, U5: Vendor (none) -> Digi-Key
Connections:
- net +5V: now also R32.1; no longer C5.2, C6.2, U3.1 (VCC), U3.14 (AFE_EN), U3.16 (LNA_EN)
- net EP: now also C6.2; no longer C6.1
- new net: C5.2, C6.1, R32.2, U3.1 (VCC), U3.14 (AFE_EN), U3.16 (LNA_EN)
Other:
- note removed: "TODO RC filter for supply"
- note removed: "TODO bipolar capable zero crossover opamp"
- moved on the sheet: C5

Commit message: w
Parts:
- renumbered C6 to C79, C5 to C80, C4 to C81, C10 to C82, C11 to C83, C12 to C84, C9 to C85, C7 to C86, C8 to C87, LS2 to LS25, R32 to R2, R5 to R3, R1 to R4, R4 to R5, R3 to R6, R2 to R7, U3 to U29, U5 to U30

Commit message: w
Parts:
- added C136, C142: 100nF, Capacitor_SMD:C_0603_1608Metric, symbol Device:C
- R2: footprint Resistor_SMD:R_0603_1608Metric_Pad0.98x0.95mm_HandSolder -> Resistor_SMD:R_0603_1608Metric
Connections:
- net +2.5V: now also C136.2
- net -2.5V: now also C142.1
- net EP: now also C136.1, C142.2
Other:
- moved on the sheet: C79, C80, C81, C82, C83, C84, C85, C86, C87, LS25, R2, R3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

Commit message: w
Parts:
- added D33: BAV99, Package_TO_SOT_SMD:SOT-23-3, symbol Device:D_Dual_Series_AKC_Parallel
- added R107: 100Ω, Resistor_SMD:R_0402_1005Metric, symbol Device:R_US
- C82: value 220pF -> 390pF
- LS25: value Speaker_Ultrasound -> 40kHz
- R3: value 30kΩ -> 20kΩ
Connections:
- net EP: now also D33.3 (common)
- net OUTN: now also U29.7 (BUFF); no longer U29.6 (~{BUFF})
- net OUTP: now also U29.6 (~{BUFF}); no longer U29.7 (BUFF)
- net at C79.1, C80.2, R2.2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: no longer U29.14 (AFE_EN), U29.16 (LNA_EN)
- net at C81.1: now also D33.1 (A), D33.2 (K), R107.1; no longer LS25.1
- new net: LS25.1, R107.2
- new net AFE_EN: U29.14 (AFE_EN)
- new net LNA_EN: U29.16 (LNA_EN)
Other:
- moved on the sheet: LS25
