File: test_boards/pcb/ultrasonic_phased_array_test.kicad_pcb (KiCad board)
At the start: 4 copper layers, 310 parts, among them Q1 G2003A, Q10 G2003A, Q11 G2003A, Q12 G2003A, Q13 G2003A, Q14 G2003A, Q15 G2003A, Q16 G2003A, Q17 G2003A, Q18 G2003A, Q19 G2003A, Q2 G2003A, Q20 G2003A, Q21 G2003A, Q22 G2003A, Q23 G2003A, Q24 G2003A, Q25 G2003A, Q26 G2003A, Q27 G2003A, Q28 G2003A, Q29 G2003A, Q3 G2003A, Q30 G2003A, Q31 G2003A, Q32 G2003A, Q33 G2003A, Q34 G2003A, Q35 G2003A, Q36 G2003A, Q37 G2003A, Q38 G2003A, Q39 G2003A, Q4 G2003A, Q40 G2003A, Q41 G2003A, Q42 G2003A, Q43 G2003A, Q44 G2003A, Q45 G2003A, Q46 G2003A, Q47 G2003A, Q48 G2003A, Q5 G2003A, Q6 G2003A, Q7 G2003A, Q8 G2003A, Q9 G2003A, U1 EG2131D, U10 OPA388xxDBV, U11 LOG300RGT, U12 OPA388xxDBV, U13 LOG300RGT, U14 OPA388xxDBV, U15 LOG300RGT, U16 OPA2626, U17 OPA2626, U18 EG2131D, U19 EG2131D, U2 AD7689xCP, U20 EG2131D, U21 EG2131D, U22 EG2131D, U23 EG2131D, U24 EG2131D, U25 EG2131D, U26 EG2131D, U27 EG2131D, U28 EG2131D, U29 EG2131D, U3 LOG300RGT, U30 EG2131D, U31 EG2131D, U32 EG2131D, U33 EG2131D, U34 EG2131D, U35 EG2131D, U36 EG2131D, U37 EG2131D, U38 EG2131D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

Commit message: w
Parts:
- C10: renamed from C65; moved to B.Cu
- C11: renamed from C66; moved to B.Cu
- C12: renamed from C64; moved to B.Cu
- C79: renamed from C6; moved to B.Cu
- C80: renamed from C5; moved to B.Cu
- C81: renamed from C4; moved to B.Cu
- C82: renamed from C10; moved to B.Cu
- C83: renamed from C11; moved to B.Cu
- C84: renamed from C12; moved to B.Cu
- C85: renamed from C9; moved to B.Cu
- C86: renamed from C7; moved to B.Cu
- C87: renamed from C8; moved to B.Cu
- D2, Q3, Q4: moved to B.Cu
- R2: renamed from R32; moved to B.Cu
- R3: renamed from R5; moved to B.Cu
- R4: renamed from R1; moved to B.Cu
- R5: renamed from R4; moved to B.Cu
- R6: renamed from R3; moved to B.Cu
- R7: renamed from R2; moved to B.Cu
- U29: renamed from U3; moved to B.Cu
- U30: renamed from U5; moved to B.Cu
- U6: renamed from U18; moved to B.Cu
- moved C81 317.7 mm to (277.0, 184.4)
- moved R2 317.6 mm to (277.1, 175.8), turned to -90 degrees
- moved C82 313.7 mm to (281.7, 177.3), turned to 180 degrees
- moved U29 312.8 mm to (281.2, 181.1), turned to -90 degrees
- moved C83 312.6 mm to (283.0, 184.0), turned to -90 degrees
- moved C85 312.4 mm to (283.6, 186.2), turned to -90 degrees
- moved C87 312.1 mm to (284.1, 187.7), turned to 180 degrees
- moved C80 312.0 mm to (278.5, 178.4)
- moved C84 311.1 mm to (284.4, 182.4)
- moved R3 310.7 mm to (281.7, 178.3)
- moved R7 310.2 mm to (283.1, 189.3), turned to 180 degrees
- moved C86 309.6 mm to (280.8, 184.1), turned to 180 degrees
- moved R4 309.0 mm to (283.7, 178.3)
- moved R5 308.1 mm to (284.7, 186.2), turned to 90 degrees
- moved R6 307.9 mm to (285.2, 189.3), turned to 180 degrees
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- renumbered C58 to C1, C30 to C100, C27 to C101, C28 to C102, C22 to C103, C29 to C104, C23 to C105, C34 to C106, C35 to C107, C33 to C108, C39 to C109, C36 to C110, C37 to C111, C31 to C112, C38 to C113, C32 to C114, C43 to C115, C44 to C116, C42 to C117, C48 to C118, C45 to C119, C46 to C120, C40 to C121, C47 to C122, C41 to C123, C52 to C124, C53 to C125, C51 to C126, C57 to C127, C54 to C128, C55 to C129, C68 to C13, C49 to C130, C56 to C131, C50 to C132, C69 to C14, C67 to C15, C71 to C16, C72 to C17, C70 to C18, C74 to C19, C59 to C2, C75 to C20, C73 to C21, C77 to C22, C78 to C23, C76 to C24, C80 to C25, C81 to C26, C79 to C27, C83 to C28, C84 to C29, C61 to C3, C82 to C30, C86 to C31, C87 to C32, C85 to C33, C89 to C34, C90 to C35, C88 to C36, C92 to C37, C93 to C38, C91 to C39, C62 to C4, C95 to C40, C96 to C41, C94 to C42, C98 to C43, C99 to C44, C97 to C45, C101 to C46, C102 to C47, C100 to C48, C104 to C49, C60 to C5, C105 to C50, C103 to C51, C107 to C52, C108 to C53, C106 to C54, C110 to C55, C111 to C56, C109 to C57, C113 to C58, C114 to C59, C63 to C6, C112 to C60, C116 to C61, C117 to C62, C115 to C63, C119 to C64, C120 to C65, C118 to C66, C122 to C67, C123 to C68, C121 to C69, C2 to C7, C125 to C70, C126 to C71, C124 to C72, C128 to C73, C129 to C74, C127 to C75, C131 to C76, C132 to C77, C130 to C78, C1 to C8, C16 to C88, C17 to C89, C3 to C9, C15 to C90, C21 to C91, C18 to C92, C19 to C93, C13 to C94, C20 to C95, C14 to C96, C25 to C97, C26 to C98, C24 to C99, LS16 to LS10, LS17 to LS11, LS18 to LS12, LS19 to LS13, LS20 to LS14, LS21 to LS15, LS22 to LS16, LS23 to LS17, LS24 to LS18, LS25 to LS19, LS8 to LS2, LS26 to LS20, LS27 to LS21, LS28 to LS22, LS29 to LS23, LS30 to LS24, LS2 to LS25, LS3 to LS26, LS4 to LS27, LS5 to LS28, LS6 to LS29, LS9 to LS3, LS7 to LS30, LS10 to LS4, LS11 to LS5, LS12 to LS6, LS13 to LS7, LS14 to LS8, LS15 to LS9, R9 to R10, R8 to R11, R6 to R12, R7 to R13, R34 to R14, R14 to R16, R13 to R17, R11 to R18, R12 to R19, R35 to R20, R20 to R21, R19 to R22, R18 to R23, R16 to R24, R17 to R25, R36 to R26, R25 to R27, R24 to R28, R23 to R29, R21 to R30, R22 to R31, R37 to R32, R30 to R33, R29 to R34, R28 to R35, R26 to R36, R27 to R37, R33 to R8, R10 to R9, U4 to U1, U22 to U10, U23 to U11, U24 to U12, U25 to U13, U26 to U14, U27 to U15, U28 to U16, U29 to U17, U30 to U18, U31 to U19, U16 to U2, U32 to U20, U33 to U21, U34 to U22, U35 to U23, U36 to U24, U37 to U25, U38 to U26, U39 to U27, U40 to U28, U17 to U3, U7 to U31, U6 to U32, U9 to U33, U8 to U34, U11 to U35, U10 to U36, U13 to U37, U12 to U38, U15 to U39, U2 to U4, U14 to U40, U1 to U5, U19 to U7, U20 to U8, U21 to U9
Routing:
- net Net-(Q3-G): track 0.00 -> 10.7 mm
- added copper zone on B.Cu, net Net-(D2-K)
- added copper zone on B.Cu, net Net-(Q3-S)
- added copper zone on B.Cu, net Net-(Q4-G)

Commit message: w
Parts:
- added C133: 100nF, Capacitor_SMD:C_0603_1608Metric, F.Cu at (356.7, 81.6)
- added C134: 100nF, Capacitor_SMD:C_0603_1608Metric, F.Cu at (356.7, 84.1)
- added C135: 100nF, Capacitor_SMD:C_0603_1608Metric, F.Cu at (356.7, 86.6)
- added C136: 100nF, Capacitor_SMD:C_0603_1608Metric, F.Cu at (382.1, 50.8)
- added C137: 100nF, Capacitor_SMD:C_0603_1608Metric, F.Cu at (388.1, 50.8)
- added C138: 100nF, Capacitor_SMD:C_0603_1608Metric, F.Cu at (394.1, 43.8)
- added C139: 100nF, Capacitor_SMD:C_0603_1608Metric, F.Cu at (382.1, 43.8)
- added C140: 100nF, Capacitor_SMD:C_0603_1608Metric, F.Cu at (388.1, 43.8)
- added C141: 100nF, Capacitor_SMD:C_0603_1608Metric, F.Cu at (394.1, 50.8)
- added C142: 100nF, Capacitor_SMD:C_0603_1608Metric, F.Cu at (382.1, 53.3)
- added C143: 100nF, Capacitor_SMD:C_0603_1608Metric, F.Cu at (388.1, 53.3)
- added C144: 100nF, Capacitor_SMD:C_0603_1608Metric, F.Cu at (394.1, 46.3)
- added C145: 100nF, Capacitor_SMD:C_0603_1608Metric, F.Cu at (382.1, 46.3)
- added C146: 100nF, Capacitor_SMD:C_0603_1608Metric, F.Cu at (388.1, 46.3)
- added C147: 100nF, Capacitor_SMD:C_0603_1608Metric, F.Cu at (394.1, 53.3)
- added C148: 10μF, Capacitor_SMD:C_1206_3216Metric, F.Cu at (357.5, 44.2)
- added C149: 22μF, Capacitor_SMD:C_1206_3216Metric, F.Cu at (357.5, 47.5)
- added C150: 10μF, Capacitor_SMD:C_1206_3216Metric, F.Cu at (357.5, 50.9)
- added C151: 10μF, Capacitor_SMD:C_1206_3216Metric, F.Cu at (357.5, 54.2)
- added C152: 10nF, Capacitor_SMD:C_0603_1608Metric, F.Cu at (367.9, 60.9)
- added C153: 10nF, Capacitor_SMD:C_0603_1608Metric, F.Cu at (367.9, 63.4)
- added C154: 10μF, Capacitor_SMD:C_1206_3216Metric, F.Cu at (357.5, 57.6)
- added C155: 10μF, Capacitor_SMD:C_1206_3216Metric, F.Cu at (357.5, 60.9)
- added C156: 1μF, Capacitor_SMD:C_1206_3216Metric, F.Cu at (357.5, 64.3)
- added C157: 1μF, Capacitor_SMD:C_1206_3216Metric, F.Cu at (357.5, 67.6)
- added C158: 1μF, Capacitor_SMD:C_1206_3216Metric, F.Cu at (357.5, 71.0)
- added J1: DF40C-80DP-0.4V, Connector_Hirose_DF40:Hirose_DF40C-80DP-0.4V_2x40-1MP_P0.4mm, F.Cu at (364.5, 77.6)
- added J2: Screw_Terminal_01x06, TerminalBlock_TE-Connectivity:TerminalBlock_TE_282834-6_1x06_P2.54mm_Horizontal, F.Cu at (362.9, 46.8)
- added R1: 10Ω, Resistor_SMD:R_0603_1608Metric, F.Cu at (356.7, 89.1)
- added R38: 24.3Ω, Resistor_SMD:R_0402_1005Metric, F.Cu at (371.7, 52.3)
- added R39: 10kΩ, Resistor_SMD:R_0402_1005Metric, F.Cu at (396.3, 75.5)
- added R40: 10kΩ, Resistor_SMD:R_0402_1005Metric, F.Cu at (386.5, 81.5)
- added R41: 10kΩ, Resistor_SMD:R_0402_1005Metric, F.Cu at (391.4, 81.5)
- added R42: 10kΩ, Resistor_SMD:R_0402_1005Metric, F.Cu at (386.5, 63.5)
- added R43: 10kΩ, Resistor_SMD:R_0402_1005Metric, F.Cu at (391.4, 63.5)
- added R44: 10kΩ, Resistor_SMD:R_0402_1005Metric, F.Cu at (396.3, 81.5)
- added R45: 10kΩ, Resistor_SMD:R_0402_1005Metric, F.Cu at (391.4, 87.4)
- added R46: 10kΩ, Resistor_SMD:R_0402_1005Metric, F.Cu at (381.6, 81.5)
- added R47: 10kΩ, Resistor_SMD:R_0402_1005Metric, F.Cu at (386.5, 69.5)
- added R48: 10kΩ, Resistor_SMD:R_0402_1005Metric, F.Cu at (391.4, 69.5)
- added R49: 10kΩ, Resistor_SMD:R_0402_1005Metric, F.Cu at (381.6, 87.4)
- added R50: 10kΩ, Resistor_SMD:R_0402_1005Metric, F.Cu at (386.5, 87.4)
- added R51: 10kΩ, Resistor_SMD:R_0402_1005Metric, F.Cu at (381.6, 75.5)
- added R52: 10kΩ, Resistor_SMD:R_0402_1005Metric, F.Cu at (396.3, 63.5)
- added R53: 10kΩ, Resistor_SMD:R_0402_1005Metric, F.Cu at (386.5, 57.5)
- added R54: 10kΩ, Resistor_SMD:R_0402_1005Metric, F.Cu at (396.3, 69.5)
- added R55: 10kΩ, Resistor_SMD:R_0402_1005Metric, F.Cu at (386.5, 75.5)
- added R56: 10kΩ, Resistor_SMD:R_0402_1005Metric, F.Cu at (391.4, 75.5)
- added R57: 10kΩ, Resistor_SMD:R_0402_1005Metric, F.Cu at (381.6, 69.5)
- added R58: 10kΩ, Resistor_SMD:R_0402_1005Metric, F.Cu at (396.3, 87.4)
- added R59: 10kΩ, Resistor_SMD:R_0402_1005Metric, F.Cu at (396.3, 57.5)
- added R60: 10kΩ, Resistor_SMD:R_0402_1005Metric, F.Cu at (381.6, 63.5)
- added R61: 10kΩ, Resistor_SMD:R_0402_1005Metric, F.Cu at (381.6, 57.5)
- added R62: 10kΩ, Resistor_SMD:R_0402_1005Metric, F.Cu at (391.4, 57.5)
- added R63: 10kΩ, Resistor_SMD:R_0402_1005Metric, F.Cu at (396.3, 77.5)
- added R64: 10kΩ, Resistor_SMD:R_0402_1005Metric, F.Cu at (386.5, 83.4)
- added R65: 10kΩ, Resistor_SMD:R_0402_1005Metric, F.Cu at (391.4, 83.4)
- added R66: 10kΩ, Resistor_SMD:R_0402_1005Metric, F.Cu at (386.5, 65.5)
- added R67: 10kΩ, Resistor_SMD:R_0402_1005Metric, F.Cu at (391.4, 65.5)
- added R68: 10kΩ, Resistor_SMD:R_0402_1005Metric, F.Cu at (396.3, 83.4)
- added R69: 10kΩ, Resistor_SMD:R_0402_1005Metric, F.Cu at (391.4, 89.4)
- added R70: 10kΩ, Resistor_SMD:R_0402_1005Metric, F.Cu at (381.6, 83.4)
- added R71: 10kΩ, Resistor_SMD:R_0402_1005Metric, F.Cu at (386.5, 71.5)
- added R72: 10kΩ, Resistor_SMD:R_0402_1005Metric, F.Cu at (391.4, 71.5)
- added R73: 10kΩ, Resistor_SMD:R_0402_1005Metric, F.Cu at (381.6, 89.4)
- added R74: 10kΩ, Resistor_SMD:R_0402_1005Metric, F.Cu at (386.5, 89.4)
- added R75: 10kΩ, Resistor_SMD:R_0402_1005Metric, F.Cu at (381.6, 77.5)
- added R76: 10kΩ, Resistor_SMD:R_0402_1005Metric, F.Cu at (396.3, 65.5)
- added R77: 10kΩ, Resistor_SMD:R_0402_1005Metric, F.Cu at (386.5, 59.5)
- added R78: 10kΩ, Resistor_SMD:R_0402_1005Metric, F.Cu at (396.3, 71.5)
- added R79: 10kΩ, Resistor_SMD:R_0402_1005Metric, F.Cu at (386.5, 77.5)
- added R80: 10kΩ, Resistor_SMD:R_0402_1005Metric, F.Cu at (391.4, 77.5)
- added R81: 10kΩ, Resistor_SMD:R_0402_1005Metric, F.Cu at (381.6, 71.5)
- added R82: 10kΩ, Resistor_SMD:R_0402_1005Metric, F.Cu at (396.3, 89.4)
- added R83: 10kΩ, Resistor_SMD:R_0402_1005Metric, F.Cu at (396.3, 59.5)
- added R84: 10kΩ, Resistor_SMD:R_0402_1005Metric, F.Cu at (381.6, 65.5)
- added R85: 10kΩ, Resistor_SMD:R_0402_1005Metric, F.Cu at (381.6, 59.5)
- added R86: 10kΩ, Resistor_SMD:R_0402_1005Metric, F.Cu at (391.4, 59.5)
- added R87: 25.5Ω, Resistor_SMD:R_0402_1005Metric, F.Cu at (371.7, 54.3)
- added R88: 25.5Ω, Resistor_SMD:R_0402_1005Metric, F.Cu at (371.7, 56.3)
- added R89: 24.3Ω, Resistor_SMD:R_0402_1005Metric, F.Cu at (371.7, 58.3)
- added U41: AZ1117CH-3.3, Package_TO_SOT_SMD:SOT-223-3_TabPin2, F.Cu at (365.3, 55.5)
- added U42: LT3032, Package_DFN_QFN:Linear_DE14MA, F.Cu at (363.3, 62.5)
- added U43: TPS60401DBV, Package_TO_SOT_SMD:SOT-23-5, F.Cu at (362.9, 67.7)
- C3, C4, C6: footprint Capacitor_SMD:C_1206_3216Metric -> Capacitor_SMD:C_0603_1608Metric
- R14, R2, R20, R26, R32, R8: footprint Resistor_SMD:R_0603_1608Metric_Pad0.98x0.95mm_HandSolder -> Resistor_SMD:R_0603_1608Metric
Connections:
- net /REFIN renamed Net-(U4-REFIN)
- U10 pad 2: /TX6_HIN -> /Transducer Tx 6/HIN_IN
- U10 pad 3: /TX6_~{LIN} -> /Transducer Tx 6/~{LIN_IN}
- U11 pad 2: /TX7_HIN -> /Transducer Tx 7/HIN_IN
- U11 pad 3: /TX7_~{LIN} -> /Transducer Tx 7/~{LIN_IN}
- U12 pad 2: /TX8_HIN -> /Transducer Tx 8/HIN_IN
- U12 pad 3: /TX8_~{LIN} -> /Transducer Tx 8/~{LIN_IN}
- U13 pad 2: /TX9_HIN -> /Transducer Tx 9/HIN_IN
- U13 pad 3: /TX9_~{LIN} -> /Transducer Tx 9/~{LIN_IN}
- U14 pad 2: /TX10_HIN -> /Transducer Tx 10/HIN_IN
- U14 pad 3: /TX10_~{LIN} -> /Transducer Tx 10/~{LIN_IN}
- U15 pad 2: /TX11_HIN -> /Transducer Tx 11/HIN_IN
- U15 pad 3: /TX11_~{LIN} -> /Transducer Tx 11/~{LIN_IN}
- U16 pad 2: /TX12_HIN -> /Transducer Tx 12/HIN_IN
- U16 pad 3: /TX12_~{LIN} -> /Transducer Tx 12/~{LIN_IN}
- U17 pad 2: /TX13_HIN -> /Transducer Tx 13/HIN_IN
- U17 pad 3: /TX13_~{LIN} -> /Transducer Tx 13/~{LIN_IN}
- U18 pad 2: /TX14_HIN -> /Transducer Tx 14/HIN_IN
- U18 pad 3: /TX14_~{LIN} -> /Transducer Tx 14/~{LIN_IN}
- U19 pad 2: /TX15_HIN -> /Transducer Tx 15/HIN_IN
- U19 pad 3: /TX15_~{LIN} -> /Transducer Tx 15/~{LIN_IN}
- U20 pad 2: /TX16_HIN -> /Transducer Tx 16/HIN_IN
- U20 pad 3: /TX16_~{LIN} -> /Transducer Tx 16/~{LIN_IN}
- U21 pad 2: /TX17_HIN -> /Transducer Tx 17/HIN_IN
- U21 pad 3: /TX17_~{LIN} -> /Transducer Tx 17/~{LIN_IN}
- U22 pad 2: /TX18_HIN -> /Transducer Tx 18/HIN_IN
- U22 pad 3: /TX18_~{LIN} -> /Transducer Tx 18/~{LIN_IN}
- U23 pad 2: /TX19_HIN -> /Transducer Tx 19/HIN_IN
- U23 pad 3: /TX19_~{LIN} -> /Transducer Tx 19/~{LIN_IN}
- U24 pad 2: /TX20_HIN -> /Transducer Tx 20/HIN_IN
- U24 pad 3: /TX20_~{LIN} -> /Transducer Tx 20/~{LIN_IN}
- U25 pad 2: /TX21_HIN -> /Transducer Tx 21/HIN_IN
- U25 pad 3: /TX21_~{LIN} -> /Transducer Tx 21/~{LIN_IN}
- U26 pad 2: /TX22_HIN -> /Transducer Tx 22/HIN_IN
- U26 pad 3: /TX22_~{LIN} -> /Transducer Tx 22/~{LIN_IN}
- U27 pad 2: /TX23_HIN -> /Transducer Tx 23/HIN_IN
- U27 pad 3: /TX23_~{LIN} -> /Transducer Tx 23/~{LIN_IN}
- U28 pad 2: /TX24_HIN -> /Transducer Tx 24/HIN_IN
- U28 pad 3: /TX24_~{LIN} -> /Transducer Tx 24/~{LIN_IN}
- U5 pad 2: /TX1_HIN -> /Transducer Tx 1/HIN_IN
- U5 pad 3: /TX1_~{LIN} -> /Transducer Tx 1/~{LIN_IN}
- U6 pad 2: /TX2_HIN -> /Transducer Tx 2/HIN_IN
- U6 pad 3: /TX2_~{LIN} -> /Transducer Tx 2/~{LIN_IN}
- U7 pad 2: /TX3_HIN -> /Transducer Tx 3/HIN_IN
- U7 pad 3: /TX3_~{LIN} -> /Transducer Tx 3/~{LIN_IN}
- U8 pad 2: /TX4_HIN -> /Transducer Tx 4/HIN_IN
- U8 pad 3: /TX4_~{LIN} -> /Transducer Tx 4/~{LIN_IN}
- U9 pad 2: /TX5_HIN -> /Transducer Tx 5/HIN_IN
- U9 pad 3: /TX5_~{LIN} -> /Transducer Tx 5/~{LIN_IN}
Routing:
- net /Transducer Tx 1/HIN_IN: track 0.00 -> 1.63 mm, vias 0 -> 1
- net /TX1_HIN: track 1.63 -> 0.00 mm, vias 1 -> 0
- net /Transducer Tx 1/~{LIN_IN}: track 0.00 -> 1.63 mm, vias 0 -> 1
- net /TX1_~{LIN}: track 1.63 -> 0.00 mm, vias 1 -> 0

Commit message: w
Parts:
- C136, C142: moved to B.Cu
- moved C136 171.5 mm to (277.9, 187.0), turned to 90 degrees
- moved C142 166.2 mm to (283.8, 187.3), turned to -90 degrees
- moved C85 2.71 mm to (286.3, 186.2)
- moved R6 1.66 mm to (283.7, 190.0)
- moved R7 1.66 mm to (281.6, 190.0)
- moved C87 1.60 mm to (285.7, 187.7), turned to 0 degrees
- moved R5 0.50 mm to (285.2, 186.2)
- moved C82 0.41 mm to (281.3, 177.2)
- moved R3 0.41 mm to (281.3, 178.2)
- moved R4 0.41 mm to (283.3, 178.3)
Routing:
- net Net-(U29-LNA_OUT): track 0.00 -> 10.3 mm
- net GND: track 23.9 -> 28.6 mm
- net Net-(U29-REF_RES): track 0.00 -> 2.08 mm
- net Net-(U29-OFFSET_CAP): track 0.00 -> 1.76 mm
- added copper zone on B.Cu, net Net-(C81-Pad1)
- added copper zone on B.Cu, net Net-(C83-Pad2)
- added copper zone on B.Cu, net Net-(U29-AFE_EN)
- added copper zone on B.Cu, net Net-(U29-LNA_IN)
- added copper zone on B.Cu, net Net-(U29-LOG_INP)
- added copper zone on B.Cu, net Net-(U29-LOG_OUT)
