File: test_boards/pcb/power.kicad_sch (KiCad schematic)
At the start: 0 parts

Commit message: w
Parts:
- added C148, C150, C151, C154, C155: 10μF, Capacitor_SMD:C_1206_3216Metric, symbol Device:C
- added C149: 22μF, Capacitor_SMD:C_1206_3216Metric, symbol Device:C
- added C152, C153: 10nF, Capacitor_SMD:C_0603_1608Metric, symbol Device:C
- added C156, C157, C158: 1μF, Capacitor_SMD:C_1206_3216Metric, symbol Device:C
- added J2: Screw_Terminal_01x06, TerminalBlock_TE-Connectivity:TerminalBlock_TE_282834-6_1x06_P2.54mm_Horizontal, symbol Connector:Screw_Terminal_01x06
- added R38, R89: 24.3Ω, Resistor_SMD:R_0402_1005Metric, symbol Device:R_US
- added R87, R88: 25.5Ω, Resistor_SMD:R_0402_1005Metric, symbol Device:R_US
- added U41: AZ1117CH-3.3, Package_TO_SOT_SMD:SOT-223-3_TabPin2, symbol symbols:AZ1117CH-3.3
- added U42: LT3032, Package_DFN_QFN:Linear_DE14MA, symbol Regulator_Linear:LT3032
- added U43: TPS60401DBV, Package_TO_SOT_SMD:SOT-23-5, symbol Regulator_SwitchedCapacitor:TPS60401DBV
Connections:
- net +2.5V: now also C152.2, C154.2, R87.1, U42.1 (OUTP)
- net +3.3V: now also C149.1, U41.2 (OUT)
- net +5V: now also C148.2, C150.2, C158.2, J2.2 (Pin_2), U41.3 (IN), U42.10 (~{SHDNN}), U42.12 (~{SHDNP}), U42.14 (INP), U43.2 (IN)
- net -2.5V: now also C153.2, C155.1, R88.2, U42.7 (OUTN)
- net VGD: now also J2.4 (Pin_4)
- net VSPK: now also J2.6 (Pin_6)
- new net: C150.1, C151.2, C154.1, C155.2, R38.2, R89.1, U42.4 (GND), U42.5 (GND)
- new net: C152.1, U42.3 (BYPP)
- new net: C156.1, U43.3 (C_{FLY-})
- new net: C156.2, U43.5 (C_{FLY+})
- new net: C153.1, U42.11 (BYPN)
- new net -5V: C151.1, C157.2, U42.6 (INN), U42.9 (INN), U43.1 (OUT)
- new net ADJN: R88.1, R89.2, U42.8 (ADJN)
- new net ADJP: R38.1, R87.2, U42.2 (ADJP)
- new net GND: C148.1, C149.2, C157.1, C158.1, J2.1 (Pin_1), J2.3 (Pin_3), J2.5 (Pin_5), U41.1 (GND), U43.4 (GND)

Commit message: w
Parts:
- removed U43: TPS60401DBV, Package_TO_SOT_SMD:SOT-23-5, symbol Regulator_SwitchedCapacitor:TPS60401DBV
- added C159, C160, C161, C162, C163, C164: 10μF, symbol Device:C
- added C165, C166: 470μF, symbol Device:C
- added C167, C168, C169, C170, C171, C172, C173, C174: 10μF, Capacitor_SMD:C_1206_3216Metric, symbol Device:C
- added D25: 20V, Diode_SMD:D_SMB, symbol Device:D_Zener
- added D26: 5.1V, Diode_SMD:D_SMB, symbol Device:D_Zener
- added U44: TPS60403DBV, Package_TO_SOT_SMD:SOT-23-5, symbol Regulator_SwitchedCapacitor:TPS60403DBV
- R38, R89: value 24.3Ω -> 24.3kΩ
- R87, R88: value 25.5Ω -> 25.5kΩ
Connections:
- net +5V: now also C173.2, C174.2, D26.1 (K), U44.2 (IN)
- net -5V: now also U44.1 (OUT)
- net GND: now also C150.1, C151.2, C154.1, C155.2, R38.2, R89.1, U42.4 (GND), U42.5 (GND), C159.1, C160.1, C161.1, C162.1, C163.1, C164.1, C165.1, C166.1, C167.1, C168.1, C169.1, C170.1, C171.1, C172.1, C173.1, C174.1, D25.2 (A), D26.2 (A), U44.4 (GND)
- net VGD: now also C166.2, C167.2, C168.2, C169.2, C170.2, C171.2, C172.2, D25.1 (K)
- net VSPK: now also C159.2, C160.2, C161.2, C162.2, C163.2, C164.2, C165.2
- net at C156.1: now also U44.3 (C_{FLY-})
- net at C156.2: now also U44.5 (C_{FLY+})
Other:
- note added: "VSPK 140V Max. VGD 11V-20V (12V Nom.)"
- moved on the sheet: C148, C149, J2, U41

Commit message: w
Parts:
- removed C168: 10μF, Capacitor_SMD:C_1206_3216Metric, symbol Device:C
- removed D26: 5.1V, Diode_SMD:D_SMB, symbol Device:D_Zener
- added C176: 10μF, Capacitor_SMD:C_1206_3216Metric, symbol Device:C
- added D26: SMAJ5.0A, Diode_SMD:D_SMA, symbol Diode:SMAJ5.0A
- C159, C160, C161, C162, C163, C164: footprint (none) -> Capacitor_SMD:CP_Elec_10x12.5; symbol Device:C -> Device:C_Polarized_US; Manufacturer Part Number (none) -> HU2G100M-CRG12; Vendor Digi-Key -> LCSC; Vendor Part Number (none) -> C117830
- C165, C166: footprint (none) -> Capacitor_THT:CP_Radial_D22.0mm_P10.00mm_SnapIn; symbol Device:C -> Device:C_Polarized_US; Manufacturer Part Number (none) -> KF471M20022*36A; Vendor Digi-Key -> LCSC; Vendor Part Number (none) -> C2684459
Connections:
- net +5V: now also D26.1 (A1)
- net GND: now also C159.2, C160.2, C161.2, C162.2, C163.2, C164.2, C165.2, C166.2, C167.2, C169.2, C170.2, C171.2, C172.2, C176.2, D26.2 (A2); no longer C159.1, C160.1, C161.1, C162.1, C163.1, C164.1, C165.1, C166.1, C167.1, C169.1, C170.1, C171.1, C172.1
- net VGD: now also C166.1, C167.1, C169.1, C170.1, C171.1, C172.1, C176.1; no longer C166.2, C167.2, C169.2, C170.2, C171.2, C172.2
- net VSPK: now also C159.1, C160.1, C161.1, C162.1, C163.1, C164.1, C165.1; no longer C159.2, C160.2, C161.2, C162.2, C163.2, C164.2, C165.2
Other:
- moved on the sheet: C167, C169, C170, C171, C172, D25
