File: test_boards/pcb/ultrasonic_phased_array_test.kicad_sch (KiCad schematic)
At the start: 12 parts, among them J1 DF40C-80DP-0.4V, U16 OPA2626, U17 OPA2626, U2 AD7689xCP, U4 OPA2626

Commit message: w
Parts:
- C58, C59, C60, C61, C62, C63, J1, R31, U16, U17, U2, U4: Vendor (none) -> Digi-Key

Commit message: w
Parts:
- renumbered C58 to C1, C59 to C2, C61 to C3, C62 to C4, C60 to C5, C63 to C6, R31 to R1, U4 to U1, U16 to U2, U17 to U3, U2 to U4

Commit message: w
Parts:
- added C133, C134, C135: 100nF, Capacitor_SMD:C_0603_1608Metric, symbol Device:C
- C3, C4, C6: footprint Capacitor_SMD:C_1206_3216Metric -> Capacitor_SMD:C_0603_1608Metric
- J1: footprint (none) -> Connector_Hirose_DF40:Hirose_DF40C-80DP-0.4V_2x40-1MP_P0.4mm
- R1: footprint (none) -> Resistor_SMD:R_0603_1608Metric
Connections:
- net +5V: now also C133.2, C134.2, C135.2
- net GND: now also C133.1, C134.1, C135.1
- net REFIN: no longer names the net of C6.2, U4.3 (REFIN)
Other:
- note added: "TODO 140V trace spacing"
- note removed: "TODO Reference"

Commit message: w
Parts:
- removed U4: AD7689xCP, Package_CSP:LFCSP-20-1EP_4x4mm_P0.5mm_EP2.5x2.5mm, symbol Analog_ADC:AD7689xCP
- added C175: 100nF, Capacitor_SMD:C_0603_1608Metric, symbol Device:C
- added R95: 10kΩ, Resistor_SMD:R_0402_1005Metric, symbol Device:R_US
- added U43: AD7699BCP, Package_CSP:LFCSP-20-1EP_4x4mm_P0.5mm_EP2.5x2.5mm, symbol Analog_ADC:AD7699BCP
- added U45: SN74LV1T34DBV, Package_TO_SOT_SMD:SOT-23-5, symbol Logic_LevelTranslator:SN74LV1T34DBV
Connections:
- net TX19_~{LIN} is gone; now on net TX13_HIN: J1.35 (Pin_35)
- net TX1_~{LIN} is gone; now on net TX2_HIN: J1.6 (Pin_6)
- net TX20_~{LIN} is gone; now on net TX15_HIN: J1.29 (Pin_29)
- net TX21_~{LIN} is gone; now on net TX17_HIN: J1.23 (Pin_23)
- net TX22_~{LIN} is gone; now on net TX19_HIN: J1.17 (Pin_17)
- net TX23_~{LIN} is gone; now on net TX21_HIN: J1.11 (Pin_11)
- net TX24_~{LIN} is gone; now on net TX23_HIN: J1.5 (Pin_5)
- net TX2_~{LIN} is gone; now on net TX4_HIN: J1.12 (Pin_12)
- net TX3_~{LIN} is gone; now on net TX6_HIN: J1.18 (Pin_18)
- net TX4_~{LIN} is gone; now on net TX8_HIN: J1.24 (Pin_24)
- net TX5_~{LIN} is gone; now on net TX10_HIN: J1.30 (Pin_30)
- net TX6_~{LIN} is gone; now on net TX12_HIN: J1.36 (Pin_36)
- net +3.3V: now also U43.15 (VIO)
- net +5V: now also C175.2, U45.5 (VCC)
- net ADC_CNV: now also U43.11 (CNV)
- net ADC_DIN: now also U43.12 (DIN)
- net ADC_SCK: now also U43.13 (SCK)
- net ADC_SDO: now also U43.14 (SDO)
- net GND: now also C175.1, U43.10 (COM), U43.21 (EPAD), U43.4 (GND), U43.5 (GND), U43.8 (IN6), U43.9 (IN7), U45.3 (GND)
- net TX10_HIN: no longer J1.58 (Pin_58)
- net TX11_HIN: now also J1.34 (Pin_34); no longer J1.64 (Pin_64)
- net TX12_HIN: no longer J1.70 (Pin_70)
- net TX13_HIN: no longer J1.69 (Pin_69)
- net TX14_HIN: now also J1.33 (Pin_33); no longer J1.63 (Pin_63)
- net TX15_HIN: no longer J1.57 (Pin_57)
- net TX16_HIN: now also J1.27 (Pin_27); no longer J1.51 (Pin_51)
- net TX17_HIN: no longer J1.45 (Pin_45)
- net TX18_HIN: now also J1.21 (Pin_21); no longer J1.39 (Pin_39)
- net TX19_HIN: no longer J1.33 (Pin_33)
- net TX20_HIN: now also J1.15 (Pin_15); no longer J1.27 (Pin_27)
- net TX21_HIN: no longer J1.21 (Pin_21)
- net TX22_HIN: now also J1.9 (Pin_9); no longer J1.15 (Pin_15)
- net TX23_HIN: no longer J1.9 (Pin_9)
- net TX2_HIN: no longer J1.10 (Pin_10)
- net TX3_HIN: now also J1.10 (Pin_10); no longer J1.16 (Pin_16)
- net TX4_HIN: no longer J1.22 (Pin_22)
- net TX5_HIN: now also J1.16 (Pin_16); no longer J1.28 (Pin_28)
- net TX6_HIN: no longer J1.34 (Pin_34)
- net TX7_HIN: now also J1.22 (Pin_22); no longer J1.40 (Pin_40)
- net TX8_HIN: no longer J1.46 (Pin_46)
- net TX9_HIN: now also J1.28 (Pin_28); no longer J1.52 (Pin_52)
- net at C2.2, R1.1: now also U43.1 (VDD), U43.20 (VDD)
- net at U1.1, U1.2 (-): now also U43.16 (IN0)
- net at C5.2: now also U43.2 (REF)
- net at U1.6 (-), U1.7: now also U43.17 (IN1)
- net at U2.1, U2.2 (-): now also U43.18 (IN2)
- net at U2.6 (-), U2.7: now also U43.19 (IN3)
- net at C6.2: now also U43.3 (REFIN)
- net at U3.1, U3.2 (-): now also U43.6 (IN4)
- net at U3.6 (-), U3.7: now also U43.7 (IN5)
- net TX10_~{LIN}: no longer names the net of J1.60 (Pin_60)
- net TX11_~{LIN}: no longer names the net of J1.66 (Pin_66)
- net TX12_~{LIN}: no longer names the net of J1.72 (Pin_72)
- net TX13_~{LIN}: no longer names the net of J1.71 (Pin_71)
- net TX14_~{LIN}: no longer names the net of J1.65 (Pin_65)
- net TX15_~{LIN}: no longer names the net of J1.59 (Pin_59)
- net TX16_~{LIN}: no longer names the net of J1.53 (Pin_53)
- net TX17_~{LIN}: no longer names the net of J1.47 (Pin_47)
- net TX18_~{LIN}: no longer names the net of J1.41 (Pin_41)
- net TX7_~{LIN}: no longer names the net of J1.42 (Pin_42)
- net TX8_~{LIN}: no longer names the net of J1.48 (Pin_48)
- net TX9_~{LIN}: no longer names the net of J1.54 (Pin_54)
- new net: R95.2, U45.2 (A)
- new net RX_AFE_EN: J1.40 (Pin_40), R95.1
- new net Transducer Rx 1/AFE_EN: U45.4 (Y)
- no-connect marks 8 -> 29
Other:
- sheet Transducer Rx 1 ports: added AFE_EN, LNA_EN; removed none
- sheet Transducer Rx 2 ports: added AFE_EN, LNA_EN; removed none
- sheet Transducer Rx 3 ports: added AFE_EN, LNA_EN; removed none
- sheet Transducer Rx 4 ports: added AFE_EN, LNA_EN; removed none
- sheet Transducer Rx 5 ports: added AFE_EN, LNA_EN; removed none
- sheet Transducer Rx 6 ports: added AFE_EN, LNA_EN; removed none
- note added: "TODO 140V trace spacing Separate Rx Signal path GND Change 5V zener to 5.6V or SMAJ5.0A Change bulk decoupling to aluminum polymer Footprints for everything potentially use 1N4148W for bootstrap diode Investigate Log out RC filter Investigate AFE input series resistor ADC Decoupling 10uF and 100nF on adc side of resistor Add extra copy of some circuitry for testing"
- note removed: "TODO 140V trace spacing"
- moved on the sheet: C1, C133, C134, C135, C2, C3, C4, C5, C6, J1, R1, U1A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

Commit message: w
Other:
- note added: "TODO 140V trace spacing Separate Rx Signal path GND Footprints for everything potentially use 1N4148W for bootstrap diode Investigate Log out RC filter Investigate AFE input series resistor ADC Decoupling 10uF and 100nF on adc side of resistor Add extra copy of some circuitry for testing"
- note removed: "TODO 140V trace spacing Separate Rx Signal path GND Change 5V zener to 5.6V or SMAJ5.0A Change bulk decoupling to aluminum polymer Footprints for everything potentially use 1N4148W for bootstrap diode Investigate Log out RC filter Investigate AFE input series resistor ADC Decoupling 10uF and 100nF on adc side of resistor Add extra copy of some circuitry for testing"
Changed lines of the file:
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@@
 		)
 	)
-	(text "TODO\n140V trace spacing\nSeparate Rx Signal path GND\nChange 5V zener to 5.6V or SMAJ5.0A\nChange bulk decoupling to aluminum polymer\nFootprints for everything\npotentially use 1N4148W for bootstrap diode\nInvestigate Log out RC filter\nInvestigate AFE input series resistor\nADC Decoupling 10uF and 100nF on adc side of resistor\nAdd extra copy of some circuitry for testing"
+	(text "TODO\n140V trace spacing\nSeparate Rx Signal path GND\n\nFootprints for everything\npotentially use 1N4148W for bootstrap diode\nInvestigate Log out RC filter\nInvestigate AFE input series resistor\nADC Decoupling 10uF and 100nF on adc side of resistor\nAdd extra copy of some circuitry for testing"
 		(exclude_from_sim no)
 		(at 206.756 68.58 0)
